File: ES8390-breakout.kicad_pcb (KiCad board)
At the start: 4 copper layers, 40.5 x 60 mm, 65 parts, among them CN1 1x14_P2.54mm, CN2 PJ-327A, CN3 PJ-327A, J1 PJ-603A, J2 JST_XH_B2B, J3 JST_XH_B2B, U1 TLV9062, U2 LP5907MFX-3.0, U3 ES8390, U4 MSM381ACP003_C51928212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

Commit message: add silkscreen
Other:
- board text added: "ADOUT/AD1"
- board text added: "AMP_SHDN"
- board text added: "CCLK"
- board text added: "CDATA"
- board text added: "DMIC_SCL/AD0"
- board text added: "DSDIN"
- board text added: "ES8390 Breakout Rev0.1"
- board text added: "GND"
- board text added: "Guitar-In"
- board text added: "LRCK"
- board text added: "Line-In"
- board text added: "Line-Out"
- board text added: "SCLK"
- board text added: "SPK OUTL"
- board text added: "SPK OUTR"
- board text added: "VAMP"
- board text added: "VIO"
- board text added: "VLDO"
Changed lines of the file:
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@@
 		(layer "Edge.Cuts")
 	)
+	(gr_text "VIO"
+		(at 87.376 97.536 0)
+		(layer "B.SilkS")
+		(effects
+			(font
+				(size 1 1)
+				(thickness 0.1)
+			)
+			(justify top mirror)
+		)
+	)
+	(gr_text "GND"
+		(at 87.63 72.136 0)
+		(layer "B.SilkS")
+		(effects
+			(font
+				(size 1 1)
+				(thickness 0.1)
+			)
+			(justify top mirror)
+		)
+	)
+	(gr_text "GND"
+		(at 87.63 82.55 0)
+		(layer "B.SilkS")
+		(effects
+			(font
+				(size 1 1)
+				(thickness 0.1)
+			)
+			(justify top mirror)
+		)
+	)
+	(gr_text "GND"
+		(at 87.63 105.156 0)
+		(layer "B.SilkS")
+		(effects
+			(font
+				(size 1 1)
+				(thickness 0.1)
+			)
+			(justify top mirror)
+		)
+	)
+	(gr_text "CCLK"
+		(at 88.138 79.756 0)
+		(layer "B.SilkS")
+		(effects
+			(font
+				(size 1 1)
+				(thickness 0.1)
+			)
+			(justify top mirror)
+		)
+	)
+	(gr_text "SCLK"
+		(at 88.138 84.836 0)
+		(layer "B.SilkS")
+		(effects
+			(font
+				(size 1 1)
+				(thickness 0.1)
+			)
+			(justify top mirror)
+		)
+	)
+	(gr_text "LRCK"
+		(at 88.138 89.916 0)
+		(layer "B.SilkS")
+		(effects
+			(font
+				(size 1 1)
+				(thickness 0.1)
+			)
+			(justify top mirror)
+		)
+	)
+	(gr_text "VLDO"
+		(at 88.138 100.076 0)
+		(layer "B.SilkS")
+		(effects
+			(font
+				(size 1 1)
+				(thickness 0.1)
+			)
+			(justify top mirror)
+		)
+	)
+	(gr_text "VAMP"
+		(at 88.138 102.616 0)
+		(layer "B.SilkS")
+		(effects
+			(font
+				(size 1 1)
+				(thickness 0.1)
+			)
+			(justify top mirror)
+		)
+	)
+	(gr_text "DSDIN"
+		(at 88.392 87.376 0)
+		(layer "B.SilkS")
+		(effects
+			(font
+				(size 1 1)
+				(thickness 0.1)
+			)
+			(justify top mirror)
+		)
+	)
+	(gr_text "CDATA"
+		(at 88.646 77.216 0)
+		(layer "B.SilkS")
+		(effects
+			(font
+				(size 1 1)
+				(thickness 0.1)
+			)
+			(justify top mirror)
+		)
+	)
+	(gr_text "AMP_SHDN"
+		(at 90.17 94.996 0)
+		(layer "B.SilkS")
+		(effects
+			(font
+				(size 1 1)
+				(thickness 0.1)
+			)
+			(justify top mirror)
+		)
+	)
+	(gr_text "ADOUT/AD1"
+		(at 90.424 92.456 0)
+		(layer "B.SilkS")
+		(effects
+			(font
+				(size 1 1)
+				(thickness 0.1)
+			)
+			(justify top mirror)
+		)
+	)
+	(gr_text "DMIC_SCL/AD0"
+		(at 91.694 74.676 0)
+		(layer "B.SilkS")
+		(effects
+			(font
+				(size 1 1)
+				(thickness 0.1)
+			)
+			(justify top mirror)
+		)
+	)
+	(gr_text "ES8390 Breakout\nRev0.1"
+		(at 117.856 63.246 0)
+		(layer "B.SilkS")
+		(effects
+			(font
+				(size 1.75 1.75)
+				(thickness 0.2)
+			)
+			(justify left bottom mirror)
+		)
+	)
+	(gr_text "Line-In"
+		(at 123.4 94.742 0)
+		(layer "B.SilkS")
+		(effects
+			(font
+				(size 1.75 1.75)
+				(thickness 0.2)
+			)
+			(justify left bottom mirror)
+		)
+	)
+	(gr_text "Guitar-In"
+		(at 123.444 74.422 0)
+		(layer "B.SilkS")
+		(effects
+			(font
+				(size 1.75 1.75)
+				(thickness 0.2)
+			)
+			(justify left bottom mirror)
+		)
+	)
+	(gr_text "Line-Out"
+		(at 123.444 108.458 0)
+		(layer "B.SilkS")
+		(effects
+			(font
+				(size 1.75 1.75)
+				(thickness 0.2)
+			)
+			(justify left bottom mirror)
+		)
+	)
+	(gr_text "SPK\nOUTR"
+		(at 95.8 112.4 0)
+		(layer "B.SilkS")
+		(effects
+			(font
+				(size 1.75 1.75)
+				(thickness 0.2)
+			)
+			(justify bottom mirror)
+		)
+	)
+	(gr_text "SPK\nOUTL"
+		(at 104 112.4 0)
+		(layer "B.SilkS")
+		(effects
+			(font
+				(size 1.75 1.75)
+				(thickness 0.2)
+			)
+			(justify bottom mirror)
+		)
+	)
 	(segment
 		(start 97 101.65)
@@
 		)
 		(min_thickness 0.25)
-		(fill
+		(fill yes
 			(thermal_gap 0.5)
 			(thermal_bridge_width 0.5)
@@
 		)
 		(min_thickness 0.25)
-		(fill
+		(fill yes
 			(thermal_gap 0.5)
 			(thermal_bridge_width 0.5)
@@
 		)
 		(min_thickness 0.25)
-		(fill
+		(fill yes
 			(thermal_gap 0.5)
 			(thermal_bridge_width 0.5)
@@
 		)
 		(min_thickness 0.25)
-		(fill
+		(fill yes
 			(thermal_gap 0.5)
 			(thermal_bridge_width 0.5)
@@
 		)
 		(min_thickness 0.25)
-		(fill
+		(fill yes
 			(thermal_gap 0.5)
 			(thermal_bridge_width 0.5)
@@
 		)
 		(min_thickness 0.25)
-		(fill
+		(fill yes
 			(thermal_gap 0.5)
 			(thermal_bridge_width 0.5)
