File: ES8390-breakout.kicad_pcb (KiCad board)
At the start: 4 copper layers, 40.5 x 60 mm, 65 parts, among them CN1 1x14_P2.54mm, CN2 PJ-327A, CN3 PJ-327A, J1 PJ-603A, J2 JST_XH_B2B, J3 JST_XH_B2B, U1 TLV9062, U2 LP5907MFX-3.0, U3 ES8390, U4 MSM381ACP003_C51928212, U5 MAX98306xDT

Commit message: fix silkscreen layout
Other:
- board text added: "MCLK"
Changed lines of the file:
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@@
 		(tags "capacitor")
 		(property "Reference" "C10"
-			(at 0 -5.8 0)
+			(at 0 -4.6 0)
 			(layer "F.SilkS")
 			(effects
@@
 		(tags "resistor")
 		(property "Reference" "R11"
-			(at 0 3.1 0)
+			(at 0 4.5 0)
 			(layer "F.SilkS")
 			(effects
@@
 	)
 	(gr_text "GND"
-		(at 87.63 82.55 0)
-		(layer "B.SilkS")
-		(effects
-			(font
-				(size 1 1)
-				(thickness 0.1)
-			)
-			(justify top mirror)
-		)
-	)
-	(gr_text "GND"
 		(at 87.63 105.156 0)
 		(layer "B.SilkS")
@@
 		(layer "B.SilkS")
 		(effects
+			(font
+				(size 1 1)
+				(thickness 0.1)
+			)
+			(justify top mirror)
+		)
+	)
+	(gr_text "MCLK"
+		(at 88.2 82.55 0)
+		(layer "B.SilkS")
+		(effects
